File: keypad.kicad_pcb (KiCad board)
At the start: 2 copper layers, 38 parts, among them SW1 RotaryEncoder_Switch, SW10 SW_Push_45deg, SW11 SW_Push_45deg, SW13 SW_Push_45deg, SW14 SW_Push_45deg, SW15 SW_Push_45deg, SW16 SW_Push_45deg, SW17 SW_Push_45deg, SW18 SW_Push_45deg, SW2 SW_Push_45deg, SW3 SW_Push_45deg, SW4 SW_Push_45deg, SW5 SW_Push_45deg, SW6 SW_Push_45deg, SW7 SW_Push_45deg, SW8 SW_Push_45deg, SW9 SW_Push_45deg, U1 XIAO-RP2040-DIP

Commit message: Add files via upload
Routing:
- net ROW3: track 155.7 -> 147.6 mm
Other:
- board outline added: 78.7 x 100 mm
Changed lines of the file:
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@@
 		(tags "diode")
 		(property "Reference" "D13"
-			(at 0 -1.05 90)
+			(at 3.345 -0.3 90)
 			(layer "F.SilkS")
 			(effects
@@
 		(stroke
 			(width 0.1)
-			(type default)
+			(type solid)
 		)
 		(fill no)
-		(layer "Margin")
+		(layer "Edge.Cuts")
 	)
 	(segment
@@
 	)
 	(segment
-		(start 176.5 107.36)
-		(end 164.691314 107.36)
+		(start 164.691314 107.36)
+		(end 176.65987 107.36)
 		(width 0.2)
 		(layer "F.Cu")
@@
 	)
 	(segment
-		(start 176.65987 107.36)
-		(end 176.5 107.36)
-		(width 0.2)
-		(layer "F.Cu")
-		(net 2)
-	)
-	(segment
 		(start 215 102.165)
 		(end 215 109.9)
@@
 	)
 	(segment
-		(start 227 37.755054)
-		(end 226.5 37.755054)
+		(start 226.5 37.755054)
+		(end 227.155054 37.755054)
 		(width 0.2)
 		(layer "F.Cu")
@@
 	)
 	(segment
-		(start 227.109108 37.801)
-		(end 227.155054 37.755054)
-		(width 0.2)
-		(layer "F.Cu")
-		(net 4)
-	)
-	(segment
-		(start 227 37.755054)
-		(end 227.155054 37.755054)
-		(width 0.2)
-		(layer "F.Cu")
-		(net 4)
-	)
-	(segment
 		(start 227.25 37.85)
 		(end 228.135 38.735)
@@
 	)
 	(segment
-		(start 157.800001 89.64)
-		(end 157.48 89.32)
+		(start 179.72 89.82)
+		(end 177 89.82)
 		(width 0.2)
 		(layer "F.Cu")
@@
 	)
 	(segment
-		(start 179.72 89.82)
-		(end 177 89.82)
+		(start 164.7 89.149)
+		(end 163.902314 89.149)
 		(width 0.2)
 		(layer "F.Cu")
@@
 	)
 	(segment
-		(start 157.48 89.32)
-		(end 156.6 88.439999)
+		(start 156.68 88.4)
+		(end 156.68 45.58)
 		(width 0.2)
 		(layer "F.Cu")
@@
 	)
 	(segment
-		(start 177 89.82)
-		(end 167.564816 89.82)
+		(start 160.64 89.64)
+		(end 156.17 89.64)
 		(width 0.2)
 		(layer "F.Cu")
@@
 	)
 	(segment
-		(start 160.64 89.64)
-		(end 157.800001 89.64)
+		(start 177 89.82)
+		(end 167.564816 89.82)
 		(width 0.2)
 		(layer "F.Cu")
@@
 	)
 	(segment
-		(start 163.3 90.549)
-		(end 164.7 89.149)
+		(start 181.690314 90.361)
+		(end 180.261 90.361)
 		(width 0.2)
 		(layer "F.Cu")
@@
 	)
 	(segment
-		(start 164.7 89.149)
-		(end 163.902314 89.149)
+		(start 161.361 90.361)
+		(end 160.64 89.64)
 		(width 0.2)
 		(layer "F.Cu")
@@
 	)
 	(segment
-		(start 156.6 88.439999)
-		(end 156.6 45.5)
+		(start 163.902314 89.149)
+		(end 162.690314 90.361)
 		(width 0.2)
 		(layer "F.Cu")
@@
 	)
 	(segment
-		(start 181.690314 90.361)
-		(end 180.261 90.361)
+		(start 202.055 44.3)
+		(end 212.855 33.5)
 		(width 0.2)
 		(layer "F.Cu")
@@
 	)
 	(segment
-		(start 163.902314 89.149)
-		(end 162.690314 90.361)
+		(start 156.03 89.5)
+		(end 156.03 89.05)
 		(width 0.2)
 		(layer "F.Cu")
@@
 	)
 	(segment
-		(start 156.68 88.4)
-		(end 156.68 88.599999)
+		(start 156.03 89.05)
+		(end 156.68 88.4)
 		(width 0.2)
 		(layer "F.Cu")
@@
 	)
 	(segment
-		(start 202.055 44.3)
-		(end 212.855 33.5)
+		(start 156.68 45.58)
+		(end 156.6 45.5)
 		(width 0.2)
 		(layer "F.Cu")
@@
 	)
 	(segment
-		(start 161.361 90.361)
-		(end 160.64 89.64)
+		(start 156.17 89.64)
+		(end 156.03 89.5)
 		(width 0.2)
 		(layer "F.Cu")
@@
 	)
 	(segment
-		(start 158.629001 90.549)
-		(end 163.3 90.549)
-		(width 0.2)
-		(layer "F.Cu")
-		(net 9)
-	)
-	(segment
 		(start 196 89.665)
 		(end 186.409816 89.665)
@@
 	)
 	(segment
-		(start 162.690314 90.361)
-		(end 161.361 90.361)
-		(width 0.2)
-		(layer "F.Cu")
-		(net 9)
-	)
-	(segment
-		(start 156.68 88.599999)
-		(end 158.629001 90.549)
+		(start 185.893816 89.149)
+		(end 182.902314 89.149)
 		(width 0.2)
 		(layer "F.Cu")
@@
 	)
 	(segment
-		(start 185.893816 89.149)
-		(end 182.902314 89.149)
+		(start 162.690314 90.361)
+		(end 161.361 90.361)
 		(width 0.2)
 		(layer "F.Cu")

Commit message: Add files via upload
Parts:
- D1, D10, D12, D13, D14, D15, D16, D17, D18, D19, D2, D20, D3, D4, D5, D6, D7, D8, D9: footprint Diode_SMD:D_0201_0603Metric -> Diode_SMD:D_SOD-123
- moved D17 3.06 mm to (225.5, 42.6)
- moved D7 2.71 mm to (175.4, 105.5)
- moved D16 2.06 mm to (231.5, 44.4)
- moved D5 1.49 mm to (157.7, 87.1), turned to -90 degrees
- moved D12 1.02 mm to (195.5, 51.5)
- moved D20 0.36 mm to (214.7, 101.7)
- moved D18 0.29 mm to (214.7, 51.3)
Connections:
- SW1 pad MP: (no net) -> GND
Routing:
- net ROW2: track 105.9 -> 139.6 mm, vias 2 -> 3
- net ROW3: track 147.6 -> 118.3 mm
- net GND: track 6.78 -> 30.2 mm
- net ROW4: track 175.1 -> 152.3 mm
- net ROW0: track 81.4 -> 73.4 mm
- net ROW1: track 90.4 -> 93.0 mm, vias 2 -> 4
- net Net-(D12-A): track 3.70 -> 5.10 mm
- net EC11SWA: track 11.1 -> 12.4 mm
- net Net-(D7-A): track 3.83 -> 5.13 mm
- net EC11SWB: track 5.94 -> 6.82 mm
- net Net-(D6-A): track 5.20 -> 4.41 mm
- net Net-(D19-A): track 4.84 -> 4.29 mm
- net Net-(D10-A): track 4.76 -> 4.21 mm
- net Net-(D20-A): track 5.39 -> 4.84 mm
- net Net-(D15-A): track 4.16 -> 4.71 mm
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